File: pcb/travyboard.kicad_pcb (KiCad board)
At the start: 2 copper layers, 360.2 x 95 mm, 144 parts, among them SW1 TAB, SW10 D, SW11 F, SW12 G, SW13 CTRL, SW14 Z, SW15 X, SW16 C, SW17 V, SW18 B, SW19 META, SW2 Q, SW20 MOD, SW21 SPACE, SW22 Y, SW23 U, SW24 I, SW25 O, SW26 P, SW27 BS, SW28 H, SW29 J, SW3 W, SW30 K, SW31 L, SW32 ;, SW33 ENTER, SW34 N, SW35 M, SW36 ,, SW37 ., SW38 /, SW39 SHIFT, SW4 E, SW40 META, SW41 MOD, SW42 SPACE, SW43 Vertical Encoder, SW44 Horizontal Encoder, SW45 T, SW46 G, SW47 Vertical Encoder, SW48 Horizontal Encoder, SW49 T, SW5 R, SW50 G, SW6 T, SW7 SHIFT, SW8 A, SW9 S, U1 RaspberryPi_Pico, U2 RaspberryPi_Pico

Commit message: Wire left half of pcb
Parts:
- added J1: AudioJack3, audio-jacks:PJ-399B-6A, F.Cu at (176.6, 85.4)
- added J2: AudioJack3, audio-jacks:PJ-399B-6A, F.Cu at (217.0, 85.4)
- moved SW47 5.09 mm to (231.0, 100.6)
- moved SW43 5.09 mm to (162.5, 100.6)
- moved D68 1.55 mm to (261.6, 108.6), turned to -156.12 degrees
- moved D74 1.26 mm to (280.2, 102.6), turned to -168.06 degrees
Connections:
- U1 pad 1: unconnected-(U1-GPIO0-Pad1) -> /Left Half/UART0_TX
- U1 pad 13: Net-(U1-GND-Pad13) -> /Left Half/GND
- U1 pad 17: unconnected-(U1-GPIO13-Pad17) -> /Left Half/ENCODER2_CLK
- U1 pad 18: Net-(U1-GND-Pad13) -> /Left Half/GND
- U1 pad 19: unconnected-(U1-GPIO14-Pad19) -> /Left Half/ENCODER2_DT
- U1 pad 2: unconnected-(U1-GPIO1-Pad2) -> /Left Half/UART0_RX
- U1 pad 20: unconnected-(U1-GPIO15-Pad20) -> /Left Half/ENCODER2_SW
- U1 pad 22: unconnected-(U1-GPIO17-Pad22) -> /Left Half/ENCODER1_DT
- U1 pad 23: Net-(U1-GND-Pad13) -> /Left Half/GND
- U1 pad 28: Net-(U1-GND-Pad13) -> /Left Half/GND
- U1 pad 29: /Left Half/ENCODER2_SW -> unconnected-(U1-GPIO22-Pad29)
- U1 pad 3: Net-(U1-GND-Pad13) -> /Left Half/GND
- U1 pad 31: unconnected-(U1-GPIO26_ADC0-Pad31) -> /Left Half/ENCODER1_CLK
- U1 pad 32: unconnected-(U1-GPIO27_ADC1-Pad32) -> /Left Half/ENCODER1_SW
- U1 pad 33: /Left Half/GND -> unconnected-(U1-AGND-Pad33)
- U1 pad 38: Net-(U1-GND-Pad13) -> /Left Half/GND
- U1 pad 8: Net-(U1-GND-Pad13) -> /Left Half/GND
- U2 pad 1: unconnected-(U2-GPIO0-Pad1) -> /Right Half/UART0_TX
- U2 pad 2: unconnected-(U2-GPIO1-Pad2) -> /Right Half/UART0_RX
Routing:
- net /Left Half/UART0_TX: track 0.00 -> 83.7 mm, vias 0 -> 1
- net /Left Half/3.3v: track 0.00 -> 74.6 mm, vias 0 -> 1
- net /Left Half/UART0_RX: track 0.00 -> 74.6 mm, vias 0 -> 2
- net /Left Half/ENCODER2_CLK: track 0.00 -> 51.7 mm, vias 0 -> 1
- net /Left Half/ENCODER2_DT: track 0.00 -> 47.4 mm, vias 0 -> 1
- net /Left Half/ENCODER1_SW: track 0.00 -> 34.0 mm
- net /Left Half/ENCODER1_CLK: track 0.00 -> 33.5 mm
- net /Left Half/ENCODER2_SW: track 0.00 -> 30.6 mm
- net /Left Half/COL_7: track 60.3 -> 87.6 mm
- net /Left Half/GND: track 0.00 -> 23.1 mm, vias 0 -> 6
- net /Left Half/ENCODER1_DT: track 0.00 -> 12.3 mm, vias 0 -> 1
- net Net-(D60-DOUT): track 46.0 -> 34.7 mm
- net /Left Half/5v: track 52.2 -> 58.4 mm, vias 23 -> 26
- net /Left Half/ROW_3: track 159.1 -> 165.2 mm
- net /Left Half/COL_2: track 203.9 -> 198.1 mm
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Other:
- outline, holes or cut-outs redrawn

Commit message: Switch to RP2040 chip on board
Parts:
- removed U1: RaspberryPi_Pico, Module_RaspberryPi_Pico:RaspberryPi_Pico_Common
- added C1: 100n, Capacitor_SMD:C_0402_1005Metric, F.Cu at (324.4, 101.0)
- added C10: 100n, Capacitor_SMD:C_0402_1005Metric, F.Cu at (330.2, 103.0)
- added C11: 100n, Capacitor_SMD:C_0402_1005Metric, F.Cu at (330.2, 105.0)
- added C12: 10u, Capacitor_SMD:C_0402_1005Metric, F.Cu at (330.2, 106.9)
- added C13: 10u, Capacitor_SMD:C_0402_1005Metric, F.Cu at (333.0, 101.0)
- added C14: 1u, Capacitor_SMD:C_0402_1005Metric, F.Cu at (333.0, 103.0)
- added C15: 27p, Capacitor_SMD:C_0402_1005Metric, F.Cu at (333.0, 105.0)
- added C16: 27p, Capacitor_SMD:C_0402_1005Metric, F.Cu at (333.0, 106.9)
- added C17: 1u, Capacitor_SMD:C_0402_1005Metric, B.Cu at (132.8, 76.6)
- added C18: 10u, Capacitor_SMD:C_0402_1005Metric, B.Cu at (164.0, 38.4)
- added C19: 10u, Capacitor_SMD:C_0402_1005Metric, B.Cu at (164.0, 39.6)
- added C2: 1u, Capacitor_SMD:C_0402_1005Metric, F.Cu at (324.4, 103.0)
- added C20: 27p, Capacitor_SMD:C_0402_1005Metric, B.Cu at (140.8, 93.5)
- added C21: 27p, Capacitor_SMD:C_0402_1005Metric, B.Cu at (140.8, 91.7)
- added C22: 100n, Capacitor_SMD:C_0402_1005Metric, B.Cu at (131.9, 90.2)
- added C23: 100n, Capacitor_SMD:C_0402_1005Metric, B.Cu at (131.9, 91.4)
- added C24: 1u, Capacitor_SMD:C_0402_1005Metric, B.Cu at (130.4, 79.2)
- added C25: 1u, Capacitor_SMD:C_0402_1005Metric, B.Cu at (129.2, 79.2)
- added C26: 100n, Capacitor_SMD:C_0402_1005Metric, B.Cu at (140.5, 87.0)
- added C27: 100n, Capacitor_SMD:C_0402_1005Metric, B.Cu at (142.0, 87.0)
- added C28: 100n, Capacitor_SMD:C_0402_1005Metric, B.Cu at (143.5, 87.0)
- added C29: 100n, Capacitor_SMD:C_0402_1005Metric, B.Cu at (145.0, 87.0)
- added C3: 100n, Capacitor_SMD:C_0402_1005Metric, F.Cu at (324.4, 105.0)
- added C30: 100n, Capacitor_SMD:C_0402_1005Metric, B.Cu at (142.0, 84.8)
- added C31: 100n, Capacitor_SMD:C_0402_1005Metric, B.Cu at (143.5, 84.8)
- added C32: 100n, Capacitor_SMD:C_0402_1005Metric, B.Cu at (145.0, 84.8)
- added C4: 1u, Capacitor_SMD:C_0402_1005Metric, F.Cu at (324.4, 106.9)
- added C5: 100n, Capacitor_SMD:C_0402_1005Metric, F.Cu at (327.3, 101.0)
- added C6: 100n, Capacitor_SMD:C_0402_1005Metric, F.Cu at (327.3, 103.0)
- added C7: 100n, Capacitor_SMD:C_0402_1005Metric, F.Cu at (327.3, 105.0)
- added C8: 100n, Capacitor_SMD:C_0402_1005Metric, F.Cu at (327.3, 106.9)
- added C9: 100n, Capacitor_SMD:C_0402_1005Metric, F.Cu at (330.2, 101.0)
- added D93: D, Diode_SMD:D_SOD-523, F.Cu at (342.8, 118.5)
- added D94: D, Diode_SMD:D_SOD-523, B.Cu at (157.2, 34.8)
- added J3: USB_C_Receptacle_USB2.0_16P, usbc:TYPE-C-31-M-13C, F.Cu at (234.6, 27.4)
- added J4: USB_C_Receptacle_USB2.0_16P, usbc:TYPE-C-31-M-13C, F.Cu at (158.9, 27.5)
- added OL1: OLED, oled:SSD1306-0.91-OLED-4pin-128x32, F.Cu at (165.4, 34.1)
- added OL2: OLED, oled:SSD1306-0.91-OLED-4pin-128x32, F.Cu at (240.4, 34.1)
- added R1: 5.1k, Resistor_SMD:R_0402_1005Metric, F.Cu at (324.4, 117.2)
- added R10: 1k, Resistor_SMD:R_0402_1005Metric, B.Cu at (135.7, 68.8)
- added R11: 10k, Resistor_SMD:R_0402_1005Metric, B.Cu at (134.2, 68.8)
- added R12: 5.1k, Resistor_SMD:R_0402_1005Metric, B.Cu at (164.0, 36.0)
- added R13: 5.1k, Resistor_SMD:R_0402_1005Metric, B.Cu at (164.0, 37.2)
- added R14: 5.6k, Resistor_SMD:R_0402_1005Metric, B.Cu at (161.6, 40.8)
- added R15: 10k, Resistor_SMD:R_0402_1005Metric, B.Cu at (164.0, 40.8)
- added R16: 1k, Resistor_SMD:R_0402_1005Metric, B.Cu at (133.6, 91.1)
- added R17: 27, Resistor_SMD:R_0402_1005Metric, B.Cu at (132.8, 79.2)
- added R18: 27, Resistor_SMD:R_0402_1005Metric, B.Cu at (131.6, 79.2)
- added R2: 5.1k, Resistor_SMD:R_0402_1005Metric, F.Cu at (324.4, 119.2)
- added R3: 5.6k, Resistor_SMD:R_0402_1005Metric, F.Cu at (324.4, 121.2)
- added R4: 10k, Resistor_SMD:R_0402_1005Metric, F.Cu at (327.4, 117.2)
- added R5: 1k, Resistor_SMD:R_0402_1005Metric, F.Cu at (327.4, 119.2)
- added R6: 27, Resistor_SMD:R_0402_1005Metric, F.Cu at (327.4, 121.2)
- added R7: 27, Resistor_SMD:R_0402_1005Metric, F.Cu at (330.3, 117.2)
- added R8: 10k, Resistor_SMD:R_0402_1005Metric, F.Cu at (330.3, 119.2)
- added R9: 1k, Resistor_SMD:R_0402_1005Metric, F.Cu at (330.3, 121.2)
- added U3: RP2040, Package_DFN_QFN:QFN-56-1EP_7x7mm_P0.4mm_EP3.2x3.2mm, B.Cu at (257.0, 87.9)
- added U4: NCP1117-1.5_SOT223, Package_TO_SOT_SMD:SOT-223-3_TabPin2, F.Cu at (327.9, 112.1)
- added U5: TPD4E05U06DQA, Package_SON:USON-10_2.5x1.0mm_P0.5mm, F.Cu at (339.5, 119.5)
- added U6: W25Q128JVS, Package_SO:SOIC-8_5.23x5.23mm_P1.27mm, B.Cu at (256.6, 78.0)
- added U7: TPD4E05U06DQA, Package_SON:USON-10_2.5x1.0mm_P0.5mm, B.Cu at (130.6, 76.0)
- added U8: NCP1117-1.5_SOT223, Package_TO_SOT_SMD:SOT-223-3_TabPin2, B.Cu at (156.9, 40.5)
- added U9: RP2040, Package_DFN_QFN:QFN-56-1EP_7x7mm_P0.4mm_EP3.2x3.2mm, B.Cu at (134.1, 84.9)
- added Y1: Crystal_GND24, Crystal:Crystal_SMD_3225-4Pin_3.2x2.5mm, F.Cu at (335.5, 119.5)
- added Y2: Crystal_GND24, Crystal:Crystal_SMD_3225-4Pin_3.2x2.5mm, B.Cu at (136.9, 92.9)
- SW45: value T -> EX1
- SW46: value G -> EX2
- SW49: value T -> EX3
- SW50: value G -> EX4
- U2: value RaspberryPi_Pico -> W25Q128JVS; footprint Module_RaspberryPi_Pico:RaspberryPi_Pico_Common -> Package_SO:SOIC-8_5.23x5.23mm_P1.27mm
- moved U2 90.7 mm to (137.5, 75.0), turned to -90 degrees
- moved J1 9.39 mm to (167.6, 82.7)
- moved SW43 6.66 mm to (156.6, 97.6)
Connections:
- D1 pad 2: /Left Half/ROW_1 -> /Left Half/ROW_0
- D10 pad 2: /Left Half/ROW_2 -> /Left Half/ROW_1
- D11 pad 2: /Left Half/ROW_2 -> /Left Half/ROW_1
- D12 pad 2: /Left Half/ROW_2 -> /Left Half/ROW_1
- D13 pad 2: /Left Half/ROW_3 -> /Left Half/ROW_2
- D14 pad 2: /Left Half/ROW_3 -> /Left Half/ROW_2
- D15 pad 2: /Left Half/ROW_3 -> /Left Half/ROW_2
- D16 pad 2: /Left Half/ROW_3 -> /Left Half/ROW_2
- D17 pad 2: /Left Half/ROW_3 -> /Left Half/ROW_2
- D18 pad 2: /Left Half/ROW_3 -> /Left Half/ROW_2
- D19 pad 2: /Right Half/ROW_1 -> /Right Half/ROW_0
- D2 pad 2: /Left Half/ROW_1 -> /Left Half/ROW_0
- D20 pad 2: /Right Half/ROW_1 -> /Right Half/ROW_0
- D21 pad 2: /Right Half/ROW_1 -> /Right Half/ROW_0
- D22 pad 2: /Right Half/ROW_1 -> /Right Half/ROW_0
- D23 pad 2: /Right Half/ROW_1 -> /Right Half/ROW_0
- D24 pad 2: /Right Half/ROW_1 -> /Right Half/ROW_0
- D25 pad 2: /Right Half/ROW_2 -> /Right Half/ROW_1
- D26 pad 2: /Right Half/ROW_2 -> /Right Half/ROW_1
- D27 pad 2: /Right Half/ROW_2 -> /Right Half/ROW_1
- D28 pad 2: /Right Half/ROW_2 -> /Right Half/ROW_1
- D29 pad 2: /Right Half/ROW_2 -> /Right Half/ROW_1
- D3 pad 2: /Left Half/ROW_1 -> /Left Half/ROW_0
- D30 pad 2: /Right Half/ROW_2 -> /Right Half/ROW_1
- D31 pad 2: /Right Half/ROW_3 -> /Right Half/ROW_2
- D32 pad 2: /Right Half/ROW_3 -> /Right Half/ROW_2
- D33 pad 2: /Right Half/ROW_3 -> /Right Half/ROW_2
- D34 pad 2: /Right Half/ROW_3 -> /Right Half/ROW_2
- D35 pad 2: /Right Half/ROW_3 -> /Right Half/ROW_2
- D36 pad 2: /Right Half/ROW_3 -> /Right Half/ROW_2
- D37 pad 2: /Left Half/ROW_4 -> /Left Half/ROW_3
- D38 pad 2: /Left Half/ROW_4 -> /Left Half/ROW_3
- D39 pad 2: /Left Half/ROW_4 -> /Left Half/ROW_3
- D4 pad 2: /Left Half/ROW_1 -> /Left Half/ROW_0
- D40 pad 2: /Right Half/ROW_4 -> /Right Half/ROW_3
- D41 pad 2: /Right Half/ROW_4 -> /Right Half/ROW_3
- D42 pad 2: /Right Half/ROW_4 -> /Right Half/ROW_3
- D43 pad 3: /Left Half/GND -> GND
- D44 pad 2: /Left Half/ROW_1 -> /Left Half/ROW_0
- D45 pad 2: /Left Half/ROW_2 -> /Left Half/ROW_1
- D46 pad 3: /Left Half/GND -> GND
- D47 pad 3: /Left Half/GND -> GND
- D48 pad 3: /Left Half/GND -> GND
- D49 pad 3: /Left Half/GND -> GND
- D5 pad 2: /Left Half/ROW_1 -> /Left Half/ROW_0
- D50 pad 3: /Left Half/GND -> GND
- D51 pad 3: /Left Half/GND -> GND
- D52 pad 3: /Left Half/GND -> GND
- D53 pad 3: /Left Half/GND -> GND
- D54 pad 3: /Left Half/GND -> GND
- D55 pad 3: /Left Half/GND -> GND
- D56 pad 3: /Left Half/GND -> GND
- D57 pad 3: /Left Half/GND -> GND
- D58 pad 3: /Left Half/GND -> GND
- D59 pad 3: /Left Half/GND -> GND
- D6 pad 2: /Left Half/ROW_1 -> /Left Half/ROW_0
- D60 pad 3: /Left Half/GND -> GND
- D61 pad 3: /Left Half/GND -> GND
- D62 pad 3: /Left Half/GND -> GND
- D63 pad 3: /Left Half/GND -> GND
- D64 pad 3: /Left Half/GND -> GND
- D65 pad 3: /Left Half/GND -> GND
- D66 pad 3: /Left Half/GND -> GND
- D67 pad 3: /Left Half/GND -> GND
- D7 pad 2: /Left Half/ROW_2 -> /Left Half/ROW_1
- D8 pad 2: /Left Half/ROW_2 -> /Left Half/ROW_1
- D9 pad 2: /Left Half/ROW_2 -> /Left Half/ROW_1
- D91 pad 2: /Right Half/ROW_1 -> /Right Half/ROW_0
- D92 pad 2: /Right Half/ROW_2 -> /Right Half/ROW_1
- J1 pad R: /Left Half/UART0_TX -> /Left Half/TX
- J1 pad S: /Left Half/GND -> GND
- J1 pad T: /Left Half/UART0_RX -> /Left Half/5v
- J2 pad T: /Right Half/UART0_TX -> /Right Half/5v
- SW1 pad 2: /Left Half/COL_1 -> /Left Half/COL_0
- SW10 pad 2: /Left Half/COL_4 -> /Left Half/COL_3
- SW11 pad 2: /Left Half/COL_5 -> /Left Half/COL_4
- SW12 pad 2: /Left Half/COL_6 -> /Left Half/COL_5
- SW13 pad 2: /Left Half/COL_1 -> /Left Half/COL_0
- SW14 pad 2: /Left Half/COL_2 -> /Left Half/COL_1
- SW15 pad 2: /Left Half/COL_3 -> /Left Half/COL_2
- SW16 pad 2: /Left Half/COL_4 -> /Left Half/COL_3
- SW17 pad 2: /Left Half/COL_5 -> /Left Half/COL_4
- SW18 pad 2: /Left Half/COL_6 -> /Left Half/COL_5
- SW19 pad 2: /Left Half/COL_4 -> /Left Half/COL_3
- SW2 pad 2: /Left Half/COL_2 -> /Left Half/COL_1
- SW20 pad 2: /Left Half/COL_5 -> /Left Half/COL_4
- SW21 pad 2: /Left Half/COL_6 -> /Left Half/COL_5
- SW3 pad 2: /Left Half/COL_3 -> /Left Half/COL_2
- SW35 pad 2: /Right Half/COL_2 -> unconnected-(SW35-Pad2)
- SW36 pad 2: /Right Half/COL_3 -> unconnected-(SW36-Pad2)
- SW37 pad 2: /Right Half/COL_4 -> unconnected-(SW37-Pad2)
- SW38 pad 2: /Right Half/COL_5 -> unconnected-(SW38-Pad2)
- SW39 pad 2: /Right Half/COL_6 -> unconnected-(SW39-Pad2)
- SW4 pad 2: /Left Half/COL_4 -> /Left Half/COL_3
- SW43 pad C: /Left Half/GND -> GND
- SW44 pad C: /Left Half/GND -> GND
- SW45 pad 2: /Left Half/COL_7 -> /Left Half/COL_6
- SW46 pad 2: /Left Half/COL_7 -> /Left Half/COL_6
- SW49 pad 2: /Right Half/COL_7 -> /Right Half/COL_0
- SW5 pad 2: /Left Half/COL_5 -> /Left Half/COL_4
- SW50 pad 2: /Right Half/COL_7 -> /Right Half/COL_0
- SW6 pad 2: /Left Half/COL_6 -> /Left Half/COL_5
- SW7 pad 2: /Left Half/COL_1 -> /Left Half/COL_0
- SW8 pad 2: /Left Half/COL_2 -> /Left Half/COL_1
- SW9 pad 2: /Left Half/COL_3 -> /Left Half/COL_2
- U2 pad 1: /Right Half/UART0_TX -> /Left Half/Left Pico/QSPI_SS
- U2 pad 2: /Right Half/UART0_RX -> /Left Half/Left Pico/QSPI_SD1
- U2 pad 3: Net-(U2-GND-Pad13) -> /Left Half/Left Pico/QSPI_SD2
- U2 pad 4: /Right Half/ROW_1 -> GND
- U2 pad 5: /Right Half/ROW_2 -> /Left Half/Left Pico/QSPI_SD0
- U2 pad 6: /Right Half/ROW_3 -> /Left Half/Left Pico/QSPI_SCLK
- U2 pad 7: /Right Half/ROW_4 -> /Left Half/Left Pico/QSPI_SD3
- U2 pad 8: Net-(U2-GND-Pad13) -> +3V3
Routing:
- net /Left Half/COL_1: track 217.3 -> 0.00 mm, vias 3 -> 0
- net /Left Half/COL_2: track 198.1 -> 0.00 mm, vias 3 -> 0
- net /Left Half/COL_4: track 188.9 -> 0.00 mm, vias 4 -> 0
- net /Left Half/COL_3: track 180.1 -> 0.00 mm, vias 3 -> 0
- net /Left Half/ROW_1: track 180.0 -> 0.00 mm
- net /Left Half/COL_5: track 171.1 -> 0.00 mm, vias 4 -> 0
- net /Left Half/ROW_3: track 165.2 -> 0.00 mm
- net /Left Half/COL_6: track 160.0 -> 0.00 mm, vias 4 -> 0
- net /Left Half/ROW_2: track 159.9 -> 0.00 mm
- net /Left Half/ROW_4: track 108.7 -> 0.00 mm
- net /Left Half/COL_7: track 87.6 -> 0.00 mm, vias 2 -> 0
- net /Left Half/UART0_TX: track 83.7 -> 0.00 mm, vias 1 -> 0
- net /Left Half/3.3v: track 74.6 -> 0.00 mm, vias 1 -> 0
- net /Left Half/UART0_RX: track 74.6 -> 0.00 mm, vias 2 -> 0
- net Net-(D47-DOUT): track 62.4 -> 0.00 mm, vias 2 -> 0
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- removed copper zone on F.Cu, net /Left Half/5v
- removed copper zone on B.Cu, net /Left Half/GND
Other:
- outline, holes or cut-outs redrawn

Commit message: Various changes
Parts:
- moved J2 9.31 mm to (225.9, 82.7)
- moved SW47 6.77 mm to (236.9, 97.3)
- moved J3 0.27 mm to (234.8, 27.5)
Other:
- outline, holes or cut-outs redrawn
Changed lines of the file:
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@@
 			(at 18.5 14 90)
 			(layer "F.Fab")
+			(hide yes)
 			(effects
 				(font
@@
 	(footprint "audio-jacks:PJ-399B-6A"
 		(layer "F.Cu")
-		(at 216.951749 85.39695 90)
+		(at 225.874024 82.748368 90)
 		(tags "usb usb-c 2.0 pd")
 		(property "Reference" "J2"
@@
 			(at 18.5 14 90)
 			(layer "F.Fab")
+			(hide yes)
 			(effects
 				(font
@@
 	(footprint "usbc:TYPE-C-31-M-13C"
 		(layer "F.Cu")
-		(at 234.553322 27.400024 180)
+		(at 234.81512 27.477415 180)
 		(descr "USB Type-C receptacle for USB 2.0 and PD, http://www.krhro.com/uploads/soft/180320/1-1P320120243.pdf")
 		(tags "usb usb-c 2.0 pd")
@@
 	(footprint "encoders:PEC12R-4220F-20024"
 		(layer "F.Cu")
-		(at 230.981444 100.607897 23.88)
+		(at 236.88703 97.305086 23.88)
 		(property "Reference" "SW47"
 			(at 0 -0.499999 23.88)
@@
 	)
 	(gr_line
+		(start 218.77716 80.36712)
+		(end 227.409184 77.092904)
+		(stroke
+			(width 0.05)
+			(type default)
+		)
+		(layer "Edge.Cuts")
+	)
+	(gr_line
 		(start 337.542471 23.812521)
 		(end 320.873707 23.812521)
@@
 		(layer "Edge.Cuts")
 	)
+	(gr_arc
+		(start 227.409566 26.789085)
+		(mid 227.583929 26.368135)
+		(end 228.004879 26.193772)
+		(stroke
+			(width 0.05)
+			(type default)
+		)
+		(layer "Edge.Cuts")
+	)
 	(gr_line
 		(start 252.805707 115.666765)
@@
 		(layer "Edge.Cuts")
 	)
-	(gr_line
-		(start 216.870497 82.248122)
-		(end 230.386131 82.248122)
-		(stroke
-			(width 0.05)
-			(type default)
-		)
-		(layer "Edge.Cuts")
-	)
 	(gr_arc
 		(start 279.201797 25.003147)
@@
 	)
 	(gr_line
-		(start 213.122054 27.979711)
-		(end 213.122054 80.856873)
+		(start 227.409184 26.789085)
+		(end 227.409184 77.092904)
 		(stroke
 			(width 0.05)
@@
 		(layer "Edge.Cuts")
 	)
+	(gr_line
+		(start 216.870497 88.552809)
+		(end 218.77716 80.36712)
+		(stroke
+			(width 0.05)
+			(type default)
+		)
+		(layer "Edge.Cuts")
+	)
 	(gr_arc
 		(start 16.668764 29.765651)
@@
 	)
 	(gr_line
-		(start 214.907993 26.193772)
+		(start 228.004879 26.193772)
 		(end 278.011171 26.193773)
 		(stroke
@@
 		(layer "Edge.Cuts")
 	)
-	(gr_arc
-		(start 213.122054 27.979711)
-		(mid 213.645148 26.716867)
-		(end 214.907993 26.193772)
-		(stroke
-			(width 0.05)
-			(type default)
-		)
-		(layer "Edge.Cuts")
-	)
 	(gr_line
 		(start 54.768796 27.384399)
@@
 	)
 	(gr_line
-		(start 216.870497 88.552809)
-		(end 230.389255 88.552809)
-		(stroke
-			(width 0.05)
-			(type default)
-		)
-		(layer "Edge.Cuts")
-	)
-	(gr_line
 		(start 160.117566 110.181995)
 		(end 168.020512 92.339323)
@@
 	)
 	(gr_line
-		(start 230.389255 88.552809)
-		(end 230.386131 82.248122)
-		(stroke
-			(width 0.05)
-			(type default)
-		)
-		(layer "Edge.Cuts")
-	)
-	(gr_line
 		(start 58.340674 83.343821)
 		(end 82.153194 83.343821)
@@
 		(stroke
 			(width 0.05)
-			(type default)
-		)
-		(layer "Edge.Cuts")
-	)
-	(gr_line
-		(start 213.122054 80.856873)
-		(end 216.870497 82.248122)
-		(stroke
-			(width 0.05)
